Commit message: [tetris.urdf.xacro] add hardwareInterface to joint

File: tetris_description/urdf/tetris.urdf.xacro (robot description, xacro)
@@ -113,17 +113,16 @@
   <transmission name="right_wheel_trans">
     <type>transmission_interface/SimpleTransmission</type>
-    <joint name="right_wheel_joint"/>
+    <joint name="right_wheel_joint">
+      <hardwareInterface>EffortJointInterface</hardwareInterface>
+    </joint>
     <actuator name="right_wheel_motor">
-      <hardwareInterface>EffortJointInterface</hardwareInterface>
-      <mechanicalReduction>1</mechanicalReduction>
     </actuator>
   </transmission>
   <transmission name="right_wheel_trans">
     <type>transmission_interface/SimpleTransmission</type>
-    <type>pr2_mechanism_model/SimpleTransmission</type>
-    <joint name="left_wheel_joint"/>
+    <joint name="left_wheel_joint">
+      <hardwareInterface>EffortJointInterface</hardwareInterface>
+    </joint>
     <actuator name="left_wheel_motor">
-      <hardwareInterface>EffortJointInterface</hardwareInterface>
-      <mechanicalReduction>1</mechanicalReduction>
     </actuator>
   </transmission>
