Commit message: [tetris_description] update model parameters, not sure if this is correct

File: tetris_description/urdf/tetris.gazebo.xacro (robot description, xacro)
@@ -16,5 +16,5 @@
       <wheelSeparation>${wheel_separation}</wheelSeparation>
       <wheelDiameter>${wheel_diameter}</wheelDiameter>
-      <torque>20</torque>
+      <torque>5</torque>
       <commandTopic>/${ns}/cmd_vel</commandTopic>
       <odometryTopic>/${ns}/odom</odometryTopic>

File: tetris_description/urdf/tetris.urdf.xacro (robot description, xacro)
@@ -33,5 +33,5 @@
     </collision>
     <inertial>
-      <mass value="1.0" />
+      <mass value="10.0" />
       <inertia ixx="1.0" ixy="0.0" ixz="0.0" iyy="1.0" iyz="0.0" izz="1.0" />
     </inertial>
@@ -46,6 +46,6 @@
     <inertial>
       <origin xyz="-0.45 0 0" />
-      <mass value="0.1" />
-      <inertia ixx="0.1" ixy="0.0" ixz="0.0" iyy="0.1" iyz="0.0" izz="0.1" />
+      <mass value="5" />
+      <inertia ixx="1" ixy="0.0" ixz="0.0" iyy="1" iyz="0.0" izz="1" />
     </inertial>
   </link>

Commit message: Add kinematic parameters obtained from designers. (INCOMPLETE YET)

File: tetris_description/urdf/tetris.gazebo.xacro (robot description, xacro)
@@ -16,5 +16,6 @@
       <wheelSeparation>${wheel_separation}</wheelSeparation>
       <wheelDiameter>${wheel_diameter}</wheelDiameter>
-      <torque>5</torque>
+      <wheelTorque>0.8</wheelTorque>
+      <wheelAcceleration>0.05</wheelAcceleration>
       <commandTopic>/${ns}/cmd_vel</commandTopic>
       <odometryTopic>/${ns}/odom</odometryTopic>

File: tetris_description/urdf/tetris.urdf.xacro (robot description, xacro)
@@ -2,7 +2,10 @@
 <robot name="tetris" xmlns:xacro="http://www.ros.org/wiki/xacro">
   <xacro:property name="PI" value="3.1415926535897931"/>
+  <xacro:property name="body_mass" value="1.89"/>
   <xacro:property name="wheel_width" value="0.04"/>
   <xacro:property name="wheel_diameter" value="0.2"/>
   <xacro:property name="wheel_separation" value="0.25"/>
+  <xacro:property name="wheel_mass" value="0.425"/>
+  <xacro:property name="tail_mass" value="0.162"/>
   <xacro:property name="ns" value="tetris" />
   <!-- Import all Gazebo-customization elements, including Gazebo colors -->
@@ -33,6 +36,7 @@
     </collision>
     <inertial>
-      <mass value="10.0" />
-      <inertia ixx="1.0" ixy="0.0" ixz="0.0" iyy="1.0" iyz="0.0" izz="1.0" />
+      <origin xyz="-0.03 0 -0.04" />
+      <mass value="${body_mass}" />
+      <inertia ixx="${(1.0/12)*body_mass*(0.2*0.2+0.1*0.1)}" ixy="0.0" ixz="0.0" iyy="${(1.0/12)*body_mass*(0.2*0.2+0.1*0.1)}" iyz="0.0" izz="${(1.0/12)*body_mass*(0.2*0.2+0.2*0.2)}" />
     </inertial>
   </link>
@@ -45,6 +49,5 @@
     </collision>
     <inertial>
-      <origin xyz="-0.45 0 0" />
-      <mass value="5" />
+      <mass value="${tail_mass}" />
       <inertia ixx="1" ixy="0.0" ixz="0.0" iyy="1" iyz="0.0" izz="1" />
     </inertial>
@@ -71,6 +74,6 @@
     </collision>
     <inertial>
-      <mass value="0.01" />
-      <inertia ixx="0.001" ixy="0.0" ixz="0.0" iyy="0.001" iyz="0.0" izz="0.001" />
+      <mass value="${wheel_mass}" />
+      <inertia ixx="${(1.0/12)*wheel_mass*(3*wheel_diameter/2*wheel_diameter/2+wheel_width*wheel_width)}" ixy="0.0" ixz="0.0" iyy="${(1.0/12)*wheel_mass*(3*wheel_diameter/2*wheel_diameter/2+wheel_width*wheel_width)}" iyz="0.0" izz="${(1.0/12)*wheel_mass*(wheel_diameter/2*wheel_diameter/2)}" />
     </inertial>
   </link>
@@ -89,6 +92,6 @@
     </collision>
     <inertial>
-      <mass value="0.01" />
-      <inertia ixx="0.001" ixy="0.0" ixz="0.0" iyy="0.001" iyz="0.0" izz="0.001" />
+      <mass value="${wheel_mass}" />
+      <inertia ixx="${(1.0/12)*wheel_mass*(3*wheel_diameter/2*wheel_diameter/2+wheel_width*wheel_width)}" ixy="0.0" ixz="0.0" iyy="${(1.0/12)*wheel_mass*(3*wheel_diameter/2*wheel_diameter/2+wheel_width*wheel_width)}" iyz="0.0" izz="${(1.0/12)*wheel_mass*(wheel_diameter/2*wheel_diameter/2)}" />
     </inertial>
   </link>

Commit message: all link is rended by texture, so material is not needed

File: tetris_description/urdf/tetris.gazebo.xacro (robot description, xacro)
@@ -29,15 +29,12 @@
     <mu1>0.1</mu1>
     <mu2>0.1</mu2>
-    <material>Gazebo/Black</material>
   </gazebo>
   <gazebo reference="tail_link">
     <mu1>0.1</mu1>
     <mu2>0.1</mu2>
-    <material>Gazebo/White</material>
   </gazebo>
   <gazebo reference="right_wheel">
     <mu1>0.8</mu1>
     <mu2>0.8</mu2>
-    <material>Gazebo/Grey</material>
     <kp>100000000.0</kp>
     <kd>1.0</kd>
@@ -46,5 +43,4 @@
     <mu1>0.8</mu1>
     <mu2>0.8</mu2>
-    <material>Gazebo/Grey</material>
     <kp>100000000.0</kp>
     <kd>1.0</kd>
